Commit message: warehouse robot model + movement

File: src/warebotsim/urdf/jackal.urdf (robot description, URDF)
Before this commit: robot jackal, 14 links, 13 joints
Links:
- link chassis_link: geometry collision box size=0.42 0.31 0.184; visual mesh filename=package://warebotsim/meshes/jackal-base.stl
- link front_fender_link: geometry visual mesh filename=package://warebotsim/meshes/jackal-fender.stl
- link front_left_wheel_link: geometry collision cylinder length=0.04 radius=0.098; visual mesh filename=package://warebotsim/meshes/jackal-wheel.stl
- link front_right_wheel_link: geometry collision cylinder length=0.04 radius=0.098; visual mesh filename=package://warebotsim/meshes/jackal-wheel.stl
- link rear_fender_link: geometry visual mesh filename=package://warebotsim/meshes/jackal-fender.stl
- link rear_left_wheel_link: geometry collision cylinder length=0.04 radius=0.098; visual mesh filename=package://warebotsim/meshes/jackal-wheel.stl
- link rear_right_wheel_link: geometry collision cylinder length=0.04 radius=0.098; visual mesh filename=package://warebotsim/meshes/jackal-wheel.stl
