Commit message: added delivery points

File: src/warebotsim/urdf/warehouse.urdf (robot description, URDF)
Before this commit: robot warehouse, 7 links, 6 joints
Links:
- added link delivery_1; visual cylinder length=0.05 radius=0.25
- added link delivery_2; visual cylinder length=0.05 radius=0.25
- added link shelf_2; visual box size=1.2 0.4 2.0
Joints:
- added joint delivery_1_joint: type fixed, parent world, child delivery_1, origin xyz=-4 0 0.025
- added joint delivery_2_joint: type fixed, parent world, child delivery_2, origin xyz=-4 -2 0.025
- added joint shelf_2_joint: type fixed, parent world, child shelf_2, origin xyz=2 -2 1.0
